File: hardware/r1/pcb/anticipy_r1.kicad_sch (KiCad schematic)
At the start: 45 parts, among them J1 USB4105-GF-A, J2 BATT, J3 MOTOR, J4 TC2030-IDC-NL, Q1 2N7002, SW1 EVQ-P7C01P, U1 MDBT50Q-1MV2, U2 BQ24075RGT, U3 AP2112K-3.3, U4 USBLC6-2SC6, U5 W25Q128JVSIQ, U6 LIS2DH12TR

Commit message: hardware/r1: fit 32 MB Macronix NOR (U5) on the verified layout
U5 W25Q128JVSIQ (16 MB) -> MX25L25645GMI-08G (256 Mbit / 32 MB) in the same
SOP-8 208-mil pattern, so placement and routing are untouched: 0 DRC
violations, 0 unconnected, 0 parity issues, ERC clean (4 intentional
warnings: PDM mics sharing DATA, /WP + /HOLD tied high).

Winbond has no >16 MB part in this footprint (WSON-8 8x6 or SOIC-16 300-mil
only); the WSON attempt collided with C4/J4 and shorted copper under the old
body to the thermal pad. docs/STORAGE.md records that and the runtime math:
32 MB is 4.3 h at 16 kbps, not 16 h, so the flash stays a BLE-offload buffer
and standalone 16 h needs the r1b SPI NAND.

Firmware: 4-byte addressing above 128 Mbit (EN4B 0xB7 or 0x13/0x12/0xDC),
JEDEC ID C2 20 19.
Parts:
- removed U5: W25Q128JVSIQ, Package_SO:SOIC-8_5.3x5.3mm_P1.27mm, symbol Memory_Flash:W25Q128JVS
- added U5: MX25L25645GMI-08G, Package_SO:SOIC-8_5.3x5.3mm_P1.27mm, symbol Memory_Flash:MX25L3233FM2
Connections:
- net +3V3: now also U5.3 (~{WP}/SIO2), U5.7 (~{HOLD}/SIO3), U5.8 (VCC)
- net FLASH_CS: now also U5.1 (~{CS})
- net FLASH_MISO: now also U5.2 (SO/SIO1)
- net FLASH_MOSI: now also U5.5 (SI/SIO0)
- net FLASH_SCK: now also U5.6 (SCLK)
- net GND: now also U5.4 (GND)
Changed lines of the file:
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@@
   (global_label "+3V3" (shape passive) (at 170.18 185.42 270) (effects (font (size 1.27 1.27))))
   (global_label "GND" (shape passive) (at 170.18 193.04 90) (effects (font (size 1.27 1.27))))
-  (symbol (lib_id "Memory_Flash:W25Q128JVS") (at 210.82 198.12 0) (unit 1)
+  (symbol (lib_id "Memory_Flash:MX25L3233FM2") (at 210.82 198.12 0) (unit 1)
     (in_bom yes) (on_board yes) (dnp no)
     (property "Reference" "U5" (at 210.82 178.12 0) (effects (font (size 1.27 1.27)) ))
-    (property "Value" "W25Q128JVSIQ" (at 210.82 175.12 0) (effects (font (size 1.27 1.27)) ))
+    (property "Value" "MX25L25645GMI-08G" (at 210.82 175.12 0) (effects (font (size 1.27 1.27)) ))
     (property "Footprint" "Package_SO:SOIC-8_5.3x5.3mm_P1.27mm" (at 210.82 172.12 0) (effects (font (size 1.27 1.27)) (hide yes)))
     (property "Datasheet" "" (at 210.82 169.12 0) (effects (font (size 1.27 1.27)) (hide yes)))
-    (property "MPN" "Winbond W25Q128JVSIQ" (at 210.82 166.12 0) (effects (font (size 1.27 1.27)) (hide yes)))
+    (property "MPN" "Macronix MX25L25645GMI-08G" (at 210.82 166.12 0) (effects (font (size 1.27 1.27)) (hide yes)))
     (instances (project "anticipy_r1" (path "/" (reference "U5") (unit 1))))
   )

Commit message: hardware/r1: fix U6 part number to LIS2DHTR, add JLCPCB BOM with LCSC codes
U6 used the LGA-14 2x2 footprint and LIS2DH symbol pinout while the BOM called out LIS2DH12TR, an LGA-12 part with a different pin order (pin 2 is CS, not SDA). Placed part is now LIS2DHTR (LCSC C155670, in stock); no footprint, placement or routing change.

anticipy_r1_bom_jlcpcb.csv maps every line to an LCSC code for PCBA. U1 (Raytac MDBT50Q-1MV2) has zero JLC stock so it must be consigned or hand soldered; J4 is Tag-Connect pads with no part to place.
Parts:
- U6: value LIS2DH12TR -> LIS2DHTR; MPN ST LIS2DH12TR -> ST LIS2DHTR
Changed lines of the file:
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@@
     (in_bom yes) (on_board yes) (dnp no)
     (property "Reference" "U6" (at 280.67 178.12 0) (effects (font (size 1.27 1.27)) ))
-    (property "Value" "LIS2DH12TR" (at 280.67 175.12 0) (effects (font (size 1.27 1.27)) ))
+    (property "Value" "LIS2DHTR" (at 280.67 175.12 0) (effects (font (size 1.27 1.27)) ))
     (property "Footprint" "Package_LGA:LGA-14_2x2mm_P0.35mm_LayoutBorder3x4y" (at 280.67 172.12 0) (effects (font (size 1.27 1.27)) (hide yes)))
     (property "Datasheet" "" (at 280.67 169.12 0) (effects (font (size 1.27 1.27)) (hide yes)))
-    (property "MPN" "ST LIS2DH12TR" (at 280.67 166.12 0) (effects (font (size 1.27 1.27)) (hide yes)))
+    (property "MPN" "ST LIS2DHTR" (at 280.67 166.12 0) (effects (font (size 1.27 1.27)) (hide yes)))
     (instances (project "anticipy_r1" (path "/" (reference "U6") (unit 1))))
   )
